File: overbed_table/数码管_按钮.kicad_sch (KiCad schematic)
At the start: 29 parts, among them SW1 KH-6X6X6H-STM, SW10 KH-6X6X6H-STM, SW11 KH-6X6X6H-STM, SW12 KH-6X6X6H-STM, SW2 KH-6X6X6H-STM, SW3 KH-6X6X6H-STM, SW4 KH-6X6X6H-STM, SW5 KH-6X6X6H-STM, SW6 KH-6X6X6H-STM, SW7 KH-6X6X6H-STM, SW8 KH-6X6X6H-STM, SW9 KH-6X6X6H-STM, U3 TM1638

Commit message: 更新原理图
Connections:
- net +5V renamed 5V_IN
- net GND renamed GND_IN
- no-connect marks 5 -> 19

Commit message: 更新原理图
Parts:
- removed LED1, LED2: FJ5361BW, lcsc_footprints:C2938342_LED-SEG-TH_11P-L37_5-W19_0-P2_54-LS15_2-BL, symbol lcsc_imported:FJ5361BW
- added LED1, LED2: 30.56, lcsc_footprints:C18187_LED-SEG-TH_FJ5361AH, symbol lcsc_imported:30_56
Connections:
- net GRID1: now also LED1.12 (DIG1)
- net GRID2: now also LED1.9 (DIG2)
- net GRID3: now also LED1.8 (DIG3)
- net GRID4: now also LED2.12 (DIG1)
- net GRID5: now also LED2.9 (DIG2)
- net GRID6: now also LED2.8 (DIG3)
- net SEG1: now also LED1.11 (A), LED2.11 (A)
- net SEG2: now also LED1.7 (B), LED2.7 (B)
- net SEG3: now also LED1.4 (C), LED2.4 (C)
- net SEG4: now also LED1.2 (D), LED2.2 (D)
- net SEG5: now also LED1.1 (E), LED2.1 (E)
- net SEG6: now also LED1.10 (F), LED2.10 (F)
- net SEG7: now also LED1.5 (G), LED2.5 (G)
- net SEG8: now also LED1.3 (DP), LED2.3 (DP)

Commit message: 原理图V1.0
Parts:
- C19: renamed from C14; footprint Button_Switch_SMD:Nidec_Copal_CAS-120A -> Capacitor_SMD:C_0603_1608Metric
- C20: renamed from C15; footprint Button_Switch_SMD:Nidec_Copal_CAS-120A -> Capacitor_SMD:C_0603_1608Metric
- C21: renamed from C16; footprint Button_Switch_SMD:Nidec_Copal_CAS-120A -> Capacitor_SMD:C_0603_1608Metric
- C22: renamed from C13; footprint Button_Switch_SMD:Nidec_Copal_CAS-120A -> Capacitor_SMD:CP_Elec_6.3x7.7
- C23: renamed from C12; footprint Button_Switch_SMD:Nidec_Copal_CAS-120A -> Capacitor_SMD:C_0603_1608Metric
- LED1, LED2: value 30.56 -> FJ5361AH
- renumbered D1 to D3, D2 to D4, D3 to D5, D4 to D6, D5 to D7, D6 to D8, R5 to R11, R6 to R12, R7 to R13, SW8 to SW10, SW9 to SW11, SW11 to SW12, SW10 to SW13, SW12 to SW14, SW1 to SW3, SW5 to SW4, SW2 to SW5, SW3 to SW7, SW7 to SW8, SW4 to SW9, U3 to U12

Commit message: 更新原理图
Parts:
- C23: value 0.1uF -> 100nF
Changed lines of the file:
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@@
 			)
 		)
-		(property "Value" "0.1uF"
+		(property "Value" "100nF"
 			(at 274.32 69.8499 0)
 			(show_name no)
