File: overbed_table/RS485_PY32.kicad_sch (KiCad schematic)
At the start: 4 parts, among them U11 SP3485EN

Commit message: 原理图V1.0
Parts:
- C35: renamed from C39; footprint Package_SO:SOIC-8_3.9x4.9mm_P1.27mm -> Capacitor_SMD:C_0603_1608Metric
- renumbered U11 to U16
