File: overbed_table/TOF.kicad_sch (KiCad schematic)
At the start: 9 parts, among them U14 VL53L0CXV0DH1

Commit message: 更新原理图
Parts:
- C41: value 47uF -> 4.7uF
Changed lines of the file:
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@@
 			)
 		)
-		(property "Value" "47uF"
+		(property "Value" "4.7uF"
 			(at 60.96 140.9699 0)
 			(show_name no)

Commit message: 原理图V1.0
Parts:
- C36: renamed from C40; footprint PCM_SparkFun-Resistor:R_0603_1608Metric -> Capacitor_SMD:C_0603_1608Metric
- C37: renamed from C41; footprint PCM_SparkFun-Resistor:R_0603_1608Metric -> Capacitor_SMD:C_0603_1608Metric
- renumbered R40 to R32, R41 to R33, R39 to R34, TP14 to TP11, TP13 to TP12, TP12 to TP13, U14 to U17

Commit message: 更新原理图
Parts:
- U17: footprint Sensor_Distance:ST_VL53L1x -> OptoDevice:ST_VL53L0X
Changed lines of the file:
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@@
 			)
 		)
-		(property "Footprint" "Sensor_Distance:ST_VL53L1x"
+		(property "Footprint" "OptoDevice:ST_VL53L0X"
 			(at 151.765 115.57 0)
 			(hide yes)
