File: overbed_table/升降电机驱动.kicad_sch (KiCad schematic)
At the start: 1 part, among them U5 DRV8243PQDGQRQ1

Commit message: 更新原理图
Parts:
- removed U5: DRV8243PQDGQRQ1, lcsc_footprints:C6225655_HVSSOP-28_L7_1-W3_0-P0_50-LS4_9-BL-EP, symbol lcsc_imported:DRV8243PQDGQRQ1
- added C25, C28, C29, C30: 100nF, lcsc_footprints:C5342036_HVSSOP-28_L7_1-W3_0-P0_50-LS4_9-BL-EP, symbol Device:C
- added C26: 220uF, lcsc_footprints:C5342036_HVSSOP-28_L7_1-W3_0-P0_50-LS4_9-BL-EP, symbol Device:C
- added C27: 10nF, lcsc_footprints:C5342036_HVSSOP-28_L7_1-W3_0-P0_50-LS4_9-BL-EP, symbol Device:C
- added R14, R15: 10k, PCM_SparkFun-Resistor:R_0603_1608Metric, symbol PCM_SparkFun-Resistor:R
- added R16: 1k, PCM_SparkFun-Resistor:R_0603_1608Metric, symbol PCM_SparkFun-Resistor:R
- added R17: 4.7k, PCM_SparkFun-Resistor:R_0603_1608Metric, symbol PCM_SparkFun-Resistor:R
- added U5: DRV8243SQDGQRQ1, lcsc_footprints:C5342036_HVSSOP-28_L7_1-W3_0-P0_50-LS4_9-BL-EP, symbol lcsc_imported:DRV8243SQDGQRQ1
Connections:
- new net: R15.2, U5.24 (nSLEEP)
- new net +12V: C25.1, C26.1, U5.21 (VM), U5.22 (VM), U5.23 (VM), U5.6 (VM), U5.7 (VM), U5.8 (VM)
- new net +3V3: R14.1, R15.1, R17.1
- new net DIR: U5.3 (PH/IN2)
- new net DRVOFF: R14.2, U5.5 (DRVOFF)
- new net GND: C25.2, C26.2, C27.1, C29.1, C30.1, R16.1, U5.12 (GND), U5.13 (GND), U5.14 (GND), U5.15 (GND), U5.16 (GND), U5.17 (GND), U5.29 (EP)
- new net IPROPI: C27.2, R16.2, U5.25 (IPROPI)
- new net OUT1: C28.1, C29.2, U5.10 (OUT1), U5.11 (OUT1), U5.9 (OUT1)
- new net OUT2: C28.2, C30.2, U5.18 (OUT2), U5.19 (OUT2), U5.20 (OUT2)
- new net PWM: U5.4 (EN/IN1)
- new net SPI_CLK: U5.1 (SCLK)
- new net SPI_CS: U5.2 (nSCS)
- new net SPI_MISO: U5.27 (SDO)
- new net SPI_MOSI: U5.28 (SDI)
- new net nFAULT: R17.2, U5.26 (nFAULT)

Commit message: 更新原理图
Parts:
- removed C27: 10nF, lcsc_footprints:C5342036_HVSSOP-28_L7_1-W3_0-P0_50-LS4_9-BL-EP, symbol Device:C
- removed C28, C29, C30: 100nF, lcsc_footprints:C5342036_HVSSOP-28_L7_1-W3_0-P0_50-LS4_9-BL-EP, symbol Device:C
- removed R14, R15: 10k, PCM_SparkFun-Resistor:R_0603_1608Metric, symbol PCM_SparkFun-Resistor:R
- removed R16: 1k, PCM_SparkFun-Resistor:R_0603_1608Metric, symbol PCM_SparkFun-Resistor:R
- removed R17: 4.7k, PCM_SparkFun-Resistor:R_0603_1608Metric, symbol PCM_SparkFun-Resistor:R
- removed U5: DRV8243SQDGQRQ1, lcsc_footprints:C5342036_HVSSOP-28_L7_1-W3_0-P0_50-LS4_9-BL-EP, symbol lcsc_imported:DRV8243SQDGQRQ1
- added U5: SS6285M-SO-TP, lcsc_footprints:C5370898_SOIC-8_L4_9-W3_9-P1_27-LS6_0-BL, symbol lcsc_imported:SS6285M-SO-TP
- C26: value 220uF -> 470uF
Connections:
- net +12V: now also U5.4 (VCC)
- net GND: now also U5.3 (GND)
- net OUT1: now also U5.7 (BO), U5.8 (BO)
- net OUT2: now also U5.5 (FO), U5.6 (FO)
- new net BI: U5.1 (BI)
- new net FI: U5.2 (FI)
Other:
- moved on the sheet: C25, C26

Commit message: 原理图V1.0
Parts:
- removed C26: 470uF, lcsc_footprints:C5342036_HVSSOP-28_L7_1-W3_0-P0_50-LS4_9-BL-EP, symbol Device:C
- added C25: 470uF, Capacitor_SMD:CP_Elec_10x10.5, symbol Device:C_Polarized
- added R20, R21: 10k, PCM_SparkFun-Resistor:R_0603_1608Metric, symbol PCM_SparkFun-Resistor:R
- C24: renamed from C25; footprint lcsc_footprints:C5342036_HVSSOP-28_L7_1-W3_0-P0_50-LS4_9-BL-EP -> Capacitor_SMD:C_0603_1608Metric
- renumbered U5 to U13
Connections:
- net +12V: now also C25.1
- net BI: now also R21.2
- net FI: now also R20.2
- net GND: now also C25.2, R20.1, R21.1
