File: overbed_table/桌脚小板.kicad_sch (KiCad schematic)
At the start: 14 parts, among them CN1 KF2EDGRC-5.08-4P, CN2 DLL-5569-6AW, SW15 KH-6X6X6H-STM, U10 KF128-5.08-2P, U12 KF128-5.08-2P, U16 WAFER-XH254WZ-2A, U17 WAFER-XH254WZ-2A, U7 PY32F030K28U6TR, X3 AFA01-S05FCA-00, X4 AFA01-S05FCA-00

Commit message: 更新原理图
Parts:
- removed U16, U17: WAFER-XH254WZ-2A, lcsc_footprints:C7432691_CONN-TH_2P-P2_50_WAFER-XH254WZ-2A, symbol lcsc_imported:WAFER-XH254WZ-2A
- added C46, C47, C48: 1uF, PCM_SparkFun-Resistor:R_0603_1608Metric, symbol Device:C
- added H2: LAIL-PZ2.54-6P-L, lcsc_footprints:C54950607_CONN-TH_LAIL-PZ2_54-6P-L, symbol lcsc_imported:LAIL-PZ2_54-6P-L
- added R46, R47, R49: 10k, PCM_SparkFun-Resistor:R_0603_1608Metric, symbol PCM_SparkFun-Resistor:R
- added SW16: KH-6X6X6H-STM, lcsc_footprints:C2837532_SW-SMD_4P-L6_0-W6_0-P4_50-LS9_0_KH-6X6X6H-STM, symbol lcsc_imported:KH-6X6X6H-STM
- added TP17, TP18, TP19, TP20: 1.0mm, PCM_SparkFun-Connector:TestPoint-1.0mm, symbol PCM_SparkFun-Connector:TestPoint_1.0mm
- added U16: WAFER-XH254WZ-4A, lcsc_footprints:C7432693_CONN-TH_4P-P2_50_WAFER-XH254WZ-4A, symbol lcsc_imported:WAFER-XH254WZ-4A
- added U20, U21: WAFER-XH254WZ-2A, lcsc_footprints:C7432691_CONN-TH_2P-P2_50_WAFER-XH254WZ-2A, symbol lcsc_imported:WAFER-XH254WZ-2A
Connections:
- net 3V3 is gone; now on net +3V3: U7.1 (VCC)
- net 升降电机驱动/DIR is gone; now on net 步进驱动/INDEX: U7.8 (PA2)
- net 升降电机驱动/DRVOFF is gone; now on net TOF_XSHUT: U7.7 (PA1)
- net 升降电机驱动/IPROPI is gone; now on net BOARD_ID: U7.6 (PA0)
- net 升降电机驱动/SPI_CS is gone; now on net 步进驱动/DIAG: U7.14 (PB0)
- net 升降电机驱动/SPI_MISO is gone; now on net MOTOR_ENC_A: U7.27 (PB4)
- net 升降电机驱动/SPI_MOSI is gone; now on net MOTOR_ENC_B: U7.28 (PB5)
- net 升降电机驱动/nFAULT is gone; now on net RS485_PY32/RS485_DE: U7.17 (PB2)
- net +3V3: now also H2.1, SW16.2 (B), U16.1, U20.1, U21.1
- net BOARD_ID: no longer U7.11 (PA5)
- net GND: now also C46.2, C47.2, C48.2, H2.2, R46.2, R47.2, R49.2, U16.2
- net MOTOR_ENC_A: no longer U7.12 (PA6)
- net MOTOR_ENC_B: no longer U7.13 (PA7)
- net PUSH_BUTTON_1: now also C46.1, R46.1, U20.2
- net PUSH_BUTTON_2: now also U7.20 (PA10-OSC32IN), C47.1, R47.1, U21.2; no longer U7.10 (PA4)
- net RS485_PY32/RS485_DE: no longer U7.25 (PA15)
- net RST: now also H2.5
- net TMC_STEP: now also U7.12 (PA6); no longer U7.32 (PB8)
- net TOF_XSHUT: no longer U7.20 (PA10-OSC32IN)
- net EXT_ENC_A: now reaches U7.18 (PA8)
- net EXT_ENC_A: now also U16.3
- net EXT_ENC_B: now reaches U7.19 (PA9-OSC32OUT)
- net EXT_ENC_B: now also U16.4
- net SWDIO: now reaches U7.23 (PA13)
- net SWDIO: now also H2.3
- net SWCLK: now reaches U7.24 (PA14)
- net SWCLK: now also H2.4
- net BOOT: now reaches U7.31 (PF4-BOOT0)
- net BOOT: now also C48.1, R49.1, SW16.4 (D)
- net 升降电机驱动/PWM: no longer names the net of U7.15 (PB1)
- net 升降电机驱动/PWM: now also TP19.1
- net 升降电机驱动/SPI_CLK: no longer names the net of U7.26 (PB3)
- net 升降电机驱动/SPI_CLK: now also TP17.1
- new net: TP18.1, U7.32 (PB8)
- new net: TP20.1, U7.11 (PA5)
- new net ISP_RX: H2.6, U7.25 (PA15)
- new net MOTOR_BI: U7.10 (PA4)
- new net MOTOR_FI: U7.13 (PA7)
- no-connect marks 3 -> 4
Other:
- sheet 升降电机驱动 ports: added BI, FI; removed +3V3, DIR, DRVOFF, IPROPI, PWM, SPI_CLK, SPI_CS, SPI_MISO, SPI_MOSI, nFAULT
- moved on the sheet: C45, CN2, R42, R43, R45, SW15, X3, X4

Commit message: 原理图V1.0
Parts:
- added C46: 100nF, Capacitor_SMD:C_0603_1608Metric, symbol Device:C
- added C47: 1uF, Capacitor_SMD:C_0603_1608Metric, symbol Device:C
- added C49, C51: 1nF, Capacitor_SMD:C_0603_1608Metric, symbol Device:C
- added R45, R47, R51, R52: 100, PCM_SparkFun-Resistor:R_0603_1608Metric, symbol PCM_SparkFun-Resistor:R
- added R48, R49: 10k, PCM_SparkFun-Resistor:R_0603_1608Metric, symbol PCM_SparkFun-Resistor:R
- C44: renamed from C45; footprint PCM_SparkFun-Resistor:R_0603_1608Metric -> Capacitor_SMD:C_0603_1608Metric
- C45: renamed from C48; footprint PCM_SparkFun-Resistor:R_0603_1608Metric -> Capacitor_SMD:C_0603_1608Metric
- C48: renamed from C47; footprint PCM_SparkFun-Resistor:R_0603_1608Metric -> Capacitor_SMD:C_0603_1608Metric
- C50: renamed from C46; footprint PCM_SparkFun-Resistor:R_0603_1608Metric -> Capacitor_SMD:C_0603_1608Metric
- renumbered CN2 to CN4, CN1 to CN5, R42 to R41, R43 to R42, R45 to R43, R49 to R44, R47 to R46, R46 to R50, TP20 to TP14, TP19 to TP15, TP18 to TP16, U7 to U19, U21 to U20, U20 to U21, U16 to U22, U10 to U23, U12 to U24, X4 to X3, X3 to X4
Connections:
- net +3V3: now also C46.2, C47.2, R48.1, R49.1
- net EXT_ENC_A: now also C51.1, R49.2, R51.1; no longer U22.3
- net EXT_ENC_B: now also C49.1, R48.2, R52.1; no longer U22.4
- net GND: now also CN4.3, C46.1, C47.1, C49.2, C51.2; no longer CN4.2
- net ISP_RX: now also H2.5; no longer H2.6
- net MOTOR_ENC_A: now also R45.1; no longer CN4.3
- net MOTOR_ENC_B: now also R47.2; no longer CN4.4
- net MOTOR_OUT1: now also CN4.4; no longer CN4.5
- net RST: now also H2.6; no longer H2.5
- new net: CN4.2, R47.1
- new net: CN4.5, R45.2
- new net: R51.2, U22.3
- new net: R52.2, U22.4
Other:
- moved on the sheet: C48, C50, CN4, H2, R46, R50, U20, U21, U22
