File: overbed_table/步进驱动.kicad_sch (KiCad schematic)
At the start: 23 parts, among them U4 TMC2209-LA

Commit message: 更新原理图
Connections:
- net UART_RX: no longer names the net of R10.1, TP8.1, U4.14 (~{PD}/UART)
- net UART_TX renamed UART_TX/RX

Commit message: 原理图V1.0
Parts:
- removed C24: 100uF, Display_7Segment:HDSP-7401, symbol Device:C
- added C29: 100uF, Capacitor_SMD:CP_Elec_6.3x7.7, symbol Device:C_Polarized
- C26: renamed from C21; value C -> 100nF; footprint Display_7Segment:HDSP-7401 -> Capacitor_SMD:C_0603_1608Metric
- C27: renamed from C22; footprint Display_7Segment:HDSP-7401 -> Capacitor_SMD:C_0603_1608Metric
- C28: renamed from C23; footprint Display_7Segment:HDSP-7401 -> Capacitor_SMD:C_0603_1608Metric
- C30: renamed from C20; footprint Button_Switch_SMD:Nidec_Copal_CAS-120A -> Capacitor_SMD:C_0603_1608Metric
- C31: renamed from C18; footprint Button_Switch_SMD:Nidec_Copal_CAS-120A -> Capacitor_SMD:C_0603_1608Metric
- C32: renamed from C19; footprint (none) -> Capacitor_SMD:C_0603_1608Metric
- C33: renamed from C17; footprint Button_Switch_SMD:Nidec_Copal_CAS-120A -> Capacitor_SMD:C_0603_1608Metric
- R24: renamed from R12; footprint PCM_SparkFun-Resistor:R_0603_1608Metric -> Resistor_SMD:R_1206_3216Metric; 功率 (none) -> 0.5W
- R25: renamed from R13; footprint PCM_SparkFun-Resistor:R_0603_1608Metric -> Resistor_SMD:R_1206_3216Metric; 耐压 (none) -> 0.5W
- TP1: renamed from TP9; footprint (none) -> PCM_SparkFun-Connector:TestPoint-1.0mm
- TP10: renamed from TP5; footprint (none) -> PCM_SparkFun-Connector:TestPoint-1.0mm
- TP2: renamed from TP10; footprint (none) -> PCM_SparkFun-Connector:TestPoint-1.0mm
- TP3: renamed from TP7; footprint (none) -> PCM_SparkFun-Connector:TestPoint-1.0mm
- TP4: renamed from TP6; footprint (none) -> PCM_SparkFun-Connector:TestPoint-1.0mm
- TP5: renamed from TP8; footprint (none) -> PCM_SparkFun-Connector:TestPoint-1.0mm
- TP6: renamed from TP1; footprint (none) -> PCM_SparkFun-Connector:TestPoint-1.0mm
- TP7: renamed from TP2; footprint (none) -> PCM_SparkFun-Connector:TestPoint-1.0mm
- TP8: renamed from TP3; footprint (none) -> PCM_SparkFun-Connector:TestPoint-1.0mm
- TP9: renamed from TP4; footprint (none) -> PCM_SparkFun-Connector:TestPoint-1.0mm
- renumbered R10 to R22, R11 to R23, U4 to U14
Connections:
- net +12V: now also C29.1
- net GND: now also C29.2
