File: overbed_table/3V3_5V_转换器.kicad_sch (KiCad schematic)
At the start: 3 parts, among them Q1 BSS138

Commit message: 更新原理图
Parts:
- added Q4, Q5: BSS138, PCM_Package_TO_SOT_SMD_AKL:SOT-23, symbol PCM_Transistor_MOSFET_AKL:BSS138
- added R22, R23, R32, R33: 4.7k, PCM_SparkFun-Resistor:R_0603_1608Metric, symbol PCM_SparkFun-Resistor:R
Connections:
- net 3V3_IN: now also Q4.1 (G), Q5.1 (G), R22.1, R32.1
- net 5V_IN: now also R23.1, R33.1
- net 3V3_SIG renamed 3V3_SIG0
- net 5V_SIG renamed 5V_SIG0
- new net 3V3_SIG1: Q4.2 (S), R22.2
- new net 3V3_SIG2: Q5.2 (S), R32.2
- new net 5V_SIG1: Q4.3 (D), R23.2
- new net 5V_SIG2: Q5.3 (D), R33.2

Commit message: 原理图V1.0
Parts:
- renumbered Q4 to Q2, Q5 to Q3, R8 to R14, R22 to R15, R32 to R16, R9 to R17, R23 to R18, R33 to R19

Commit message: update: 更新ESP32 PCB
Parts:
- R14, R15, R16, R17, R18, R19: footprint PCM_SparkFun-Resistor:R_0603_1608Metric -> Resistor_SMD:R_0603_1608Metric
Changed lines of the file:
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@@
 			)
 		)
-		(property "Footprint" "PCM_SparkFun-Resistor:R_0603_1608Metric"
+		(property "Footprint" "Resistor_SMD:R_0603_1608Metric"
 			(at 113.792 76.2 0)
 			(hide yes)
@@
 			)
 		)
-		(property "Footprint" "PCM_SparkFun-Resistor:R_0603_1608Metric"
+		(property "Footprint" "Resistor_SMD:R_0603_1608Metric"
 			(at 113.792 137.16 0)
 			(hide yes)
@@
 			)
 		)
-		(property "Footprint" "PCM_SparkFun-Resistor:R_0603_1608Metric"
+		(property "Footprint" "Resistor_SMD:R_0603_1608Metric"
 			(at 158.242 76.2 0)
 			(hide yes)
@@
 			)
 		)
-		(property "Footprint" "PCM_SparkFun-Resistor:R_0603_1608Metric"
+		(property "Footprint" "Resistor_SMD:R_0603_1608Metric"
 			(at 113.792 106.68 0)
 			(hide yes)
@@
 			)
 		)
-		(property "Footprint" "PCM_SparkFun-Resistor:R_0603_1608Metric"
+		(property "Footprint" "Resistor_SMD:R_0603_1608Metric"
 			(at 158.242 106.68 0)
 			(hide yes)
@@
 			)
 		)
-		(property "Footprint" "PCM_SparkFun-Resistor:R_0603_1608Metric"
+		(property "Footprint" "Resistor_SMD:R_0603_1608Metric"
 			(at 158.242 137.16 0)
 			(hide yes)
