File: overbed_table/LED灯驱动.kicad_sch (KiCad schematic)
At the start: 3 parts, among them Q2 AON7524

Commit message: 原理图V1.0
Parts:
- renumbered Q2 to Q4, R18 to R35, R19 to R36

Commit message: update: 更新ESP32 PCB
Parts:
- R35, R36: footprint PCM_SparkFun-Resistor:R_0603_1608Metric -> Resistor_SMD:R_0603_1608Metric
Changed lines of the file:
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@@
 			)
 		)
-		(property "Footprint" "PCM_SparkFun-Resistor:R_0603_1608Metric"
+		(property "Footprint" "Resistor_SMD:R_0603_1608Metric"
 			(at 150.622 97.79 0)
 			(hide yes)
@@
 			)
 		)
-		(property "Footprint" "PCM_SparkFun-Resistor:R_0603_1608Metric"
+		(property "Footprint" "Resistor_SMD:R_0603_1608Metric"
 			(at 135.89 93.472 0)
 			(hide yes)
