File: overbed_table/RS485_ESP32.kicad_sch (KiCad schematic)
At the start: 6 parts, among them U9 SP3485EN

Commit message: 更新原理图
Parts:
- R25: value 10k -> 390
Changed lines of the file:
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@@
 			)
 		)
-		(property "Value" "10k"
+		(property "Value" "390"
 			(at 176.53 102.8699 90)
 			(show_name no)

Commit message: 原理图V1.0
Parts:
- removed C32: 100nF, Package_SO:SOIC-8_3.9x4.9mm_P1.27mm, symbol Device:C
- removed R20: 10k, PCM_SparkFun-Resistor:R_0603_1608Metric, symbol PCM_SparkFun-Resistor:R
- removed R21: 120, PCM_SparkFun-Resistor:R_0603_1608Metric, symbol PCM_SparkFun-Resistor:R
- removed U9: SP3485EN, Package_SO:SOIC-8_3.9x4.9mm_P1.27mm, symbol Interface_UART:SP3485EN
- added C34: 100nF, Capacitor_SMD:C_0603_1608Metric, symbol Device:C
- added R26: 10k, PCM_SparkFun-Resistor:R_0603_1608Metric, symbol PCM_SparkFun-Resistor:R
- added R27: 120, PCM_SparkFun-Resistor:R_0603_1608Metric, symbol PCM_SparkFun-Resistor:R
- added U15: SP3485EN, Package_SO:SOIC-8_3.9x4.9mm_P1.27mm, symbol Interface_UART:SP3485EN
- renumbered R24 to R28, R25 to R29
Connections:
- net +3V3: now also C34.1, U15.8 (VCC)
- net GND: now also C34.2, R26.2, U15.5 (GND)
- net RS485_A: now also R27.1, U15.6 (A)
- net RS485_B: now also R27.2, U15.7 (B)
- net RS485_DE: now also R26.1, U15.2 (~{RE}), U15.3 (DE)
- net RS485_RX: now also U15.1 (RO)
- net RS485_TX: now also U15.4 (DI)

Commit message: update: 更新ESP32 PCB
Parts:
- R26, R27, R28, R29: footprint PCM_SparkFun-Resistor:R_0603_1608Metric -> Resistor_SMD:R_0603_1608Metric
Connections:
- net RS485_A renamed RS485_P
- net RS485_B renamed RS485_N
Changed lines of the file:
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@@
 		)
 	)
-	(hierarchical_label "RS485_A"
+	(hierarchical_label "RS485_P"
 		(shape bidirectional)
 		(at 186.69 74.93 0)
@@
 		)
 	)
-	(hierarchical_label "RS485_B"
+	(hierarchical_label "RS485_N"
 		(shape bidirectional)
 		(at 186.69 92.71 0)
@@
 			)
 		)
-		(property "Footprint" "PCM_SparkFun-Resistor:R_0603_1608Metric"
+		(property "Footprint" "Resistor_SMD:R_0603_1608Metric"
 			(at 178.562 67.31 0)
 			(hide yes)
@@
 			)
 		)
-		(property "Footprint" "PCM_SparkFun-Resistor:R_0603_1608Metric"
+		(property "Footprint" "Resistor_SMD:R_0603_1608Metric"
 			(at 99.822 95.25 0)
 			(hide yes)
@@
 			)
 		)
-		(property "Footprint" "PCM_SparkFun-Resistor:R_0603_1608Metric"
+		(property "Footprint" "Resistor_SMD:R_0603_1608Metric"
 			(at 178.562 101.6 0)
 			(hide yes)
@@
 			)
 		)
-		(property "Footprint" "PCM_SparkFun-Resistor:R_0603_1608Metric"
+		(property "Footprint" "Resistor_SMD:R_0603_1608Metric"
 			(at 165.862 83.82 0)
 			(hide yes)
