File: overbed_table/overbed_table.kicad_pcb (KiCad board)
At the start: 4 copper layers, 105 x 90 mm, 284 parts, among them CN10 DLL-5569-2AW, CN2 KF2EDGRC-5.08-4P, CN3 KF2EDGRC-5.08-4P, CN4 DLL-5569-6AW, CN5 KF2EDGRC-5.08-4P, CN6 DLL-5569-6AW, CN7 KF2EDGRC-5.08-4P, CN8 DLL-5569-2AW, CN9 DLL-5569-2AW, Q1 BSS138, Q2 BSS138, Q3 BSS138, Q4 AON7524, Q5 AON7524, Q6 AON7524, SW1 KH-6X6X6H-STM, SW10 KH-6X6X6H-STM, SW11 KH-6X6X6H-STM, SW12 KH-6X6X6H-STM, SW13 KH-6X6X6H-STM, SW14 KH-6X6X6H-STM, SW15 KH-6X6X6H-STM, SW16 KH-6X6X6H-STM, SW17 KH-6X6X6H-STM, SW18 KH-6X6X6H-STM, SW2 KH-6X6X6H-STM, SW3 KH-6X6X6H-STM, SW4 KH-6X6X6H-STM, SW5 KH-6X6X6H-STM, SW6 KH-6X6X6H-STM, SW7 KH-6X6X6H-STM, SW8 KH-6X6X6H-STM, SW9 KH-6X6X6H-STM, U1 AP2112K-3.3TRG1, U10 TPS562201DDCR, U11 TPS562201DDCR, U12 TM1638, U13 SS6285M-SO-TP, U14 TMC2209-LA, U15 SP3485EN, U16 SP3485EN, U17 VL53L0CXV0DH1, U18 TPS562201DDCR, U19 PY32F030K28U6TR, U2 ESP32-C3-WROOM-02, U20 WAFER-XH254WZ-2A, U21 WAFER-XH254WZ-2A, U22 WAFER-XH254WZ-4A, U23 KF128-5.08-2P, U24 KF128-5.08-2P, U25 PY32F030K28U6TR, U26 WAFER-XH254WZ-2A, U27 WAFER-XH254WZ-2A, U28 WAFER-XH254WZ-4A, U29 KF128-5.08-2P, U3 WAFER-XH254WZ-2A, U30 KF128-5.08-2P, U31 TMC2209-LA, U32 VL53L0CXV0DH1, U33 TPS562201DDCR, U34 SS6285M-SO-TP, U35 SP3485EN, U4 BSMD2920-500-24V, U5 BSMD2920-500-24V, U6 BSMD2920-500-24V, U7 KF7620-7.62-2P, X1 AFA01-S05FCA-00, X2 AFA01-S05FCA-00, X3 AFA01-S05FCA-00, X4 AFA01-S05FCA-00, X5 AFA01-S05FCA-00, X6 AFA01-S05FCA-00

Commit message: update: 更新ESP32 PCB
Parts:
- removed C19, C20, C21: 100pF, Capacitor_SMD:C_0603_1608Metric
- removed C22, C29, C63: 100uF, Capacitor_SMD:CP_Elec_6.3x7.7
- removed C23, C24, C26, C27, C28, C30, C31, C35, C36, C46, C54, C60, C61, C62, C64, C65, C68, C76, C78: 100nF, Capacitor_SMD:C_0603_1608Metric
- removed C25, C77: 470uF, Capacitor_SMD:CP_Elec_10x10.5
- removed C32, C37, C66, C69: 4.7uF, Capacitor_SMD:C_0603_1608Metric
- removed C33, C67: 22nF, Capacitor_SMD:C_0603_1608Metric
- removed C38, C39, C70, C71: 10uF, Capacitor_SMD:C_0805_2012Metric
- removed C40, C72: 100nF, Capacitor_SMD:C_0805_2012Metric
- removed C41, C42, C43, C73, C74, C75: 22uF, Capacitor_SMD:C_0805_2012Metric
- removed C44, C45, C47, C48, C50, C52, C53, C55, C56, C58: 1uF, Capacitor_SMD:C_0603_1608Metric
- removed C49, C51, C57, C59: 1nF, Capacitor_SMD:C_0603_1608Metric
- removed CN4, CN6: DLL-5569-6AW, lcsc_footprints:C22365656_CONN-TH_6P-P4_20_C9900016025
- removed CN5, CN7: KF2EDGRC-5.08-4P, lcsc_footprints:C441238_CONN-TH_4P-P5_08_KF2EDGRC-5_08-4P
- removed D3, D4, D5, D6, D7, D8: 1N4148W, PCM_Diode_SMD_AKL:D_SOD-123
- removed H2, H3: LAIL-PZ2.54-6P-L, lcsc_footprints:C54950607_CONN-TH_LAIL-PZ2_54-6P-L
- removed L3, L4: FXL0630-3R3-M, lcsc_footprints:C167219_IND-SMD_L7_0-W6_6
- removed LED1, LED2: FJ5361AH, lcsc_footprints:C18187_LED-SEG-TH_FJ5361AH
- removed R11, R12, R13, R20, R21, R23, R30, R34, R40, R41, R43, R44, R46, R48, R49, R50, R53, R55, R56, R58, R60, R61, R62, R66, R71, R73, R74, R75, R76: 10k, PCM_SparkFun-Resistor:R_0603_1608Metric
- removed R22, R65: 1k, PCM_SparkFun-Resistor:R_0603_1608Metric
- removed R24, R25, R67, R68: 0.15, Resistor_SMD:R_1206_3216Metric
- removed R31, R77: 120, PCM_SparkFun-Resistor:R_0603_1608Metric
- removed R32, R33, R69, R70: 4.7k, PCM_SparkFun-Resistor:R_0603_1608Metric
- removed R39, R72: 33.2k, PCM_SparkFun-Resistor:R_0603_1608Metric
- removed R42, R54: 0, PCM_SparkFun-Resistor:R_0603_1608Metric
- removed R45, R47, R51, R52, R57, R59, R63, R64: 100, PCM_SparkFun-Resistor:R_0603_1608Metric
- removed SW10, SW11, SW12, SW13, SW14, SW15, SW16, SW17, SW18, SW3, SW4, SW5, SW6, SW7, SW8, SW9: KH-6X6X6H-STM, lcsc_footprints:C2837532_SW-SMD_4P-L6_0-W6_0-P4_50-LS9_0_KH-6X6X6H-STM
- removed TP1, TP10, TP2, TP22, TP23, TP24, TP25, TP26, TP27, TP28, TP29, TP3, TP30, TP31, TP4, TP5, TP6, TP7, TP8, TP9: TestPoint, PCM_SparkFun-Connector:TestPoint-1.0mm
- removed TP11, TP12, TP13, TP14, TP15, TP16, TP17, TP18, TP19, TP20, TP21, TP32, TP33, TP34: 1.0mm, PCM_SparkFun-Connector:TestPoint-1.0mm
- removed U12: TM1638, lcsc_footprints:C19187_SOIC-28_L17_9-W7_5-P1_27-LS10_3-BL
- removed U13, U34: SS6285M-SO-TP, lcsc_footprints:C5370898_SOIC-8_L4_9-W3_9-P1_27-LS6_0-BL
- removed U14, U31: TMC2209-LA, Package_DFN_QFN:VQFN-28-1EP_5x5mm_P0.5mm_EP3.7x3.7mm_ThermalVias
- removed U16, U35: SP3485EN, Package_SO:SOIC-8_3.9x4.9mm_P1.27mm
- removed U17, U32: VL53L0CXV0DH1, OptoDevice:ST_VL53L0X
- removed U18, U33: TPS562201DDCR, lcsc_footprints:C90061_SOT-23-6_L2_9-W1_6-P0_95-LS2_8-BR
- removed U19, U25: PY32F030K28U6TR, lcsc_footprints:C3018718_QFN-32_L5_0-W5_0-P0_50-TL-EP3_5
- removed U20, U21, U26, U27: WAFER-XH254WZ-2A, lcsc_footprints:C7432691_CONN-TH_2P-P2_50_WAFER-XH254WZ-2A
- removed U22, U28: WAFER-XH254WZ-4A, lcsc_footprints:C7432693_CONN-TH_4P-P2_50_WAFER-XH254WZ-4A
- removed U23, U24, U29, U30: KF128-5.08-2P, lcsc_footprints:C474952_CONN-TH_P5_08_KF128-5_08-2P
- removed X2, X3, X4, X5, X6: AFA01-S05FCA-00, lcsc_footprints:C262753_FPC-SMD_AFA01-S05FCA-00
- R1, R14, R15, R16, R17, R18, R19, R2, R26, R27, R28, R29, R3, R35, R36, R37, R38, R4, R5, R6, R7, R78, R79, R8, R80: footprint PCM_SparkFun-Resistor:R_0603_1608Metric -> Resistor_SMD:R_0603_1608Metric
- moved U15 222.1 mm to (53.2, 85.2), turned to -90 degrees
- moved R29 220.4 mm to (48.2, 87.4), turned to -90 degrees
- moved R28 220.3 mm to (48.2, 84.4), turned to -90 degrees
- moved R26 219.8 mm to (49.0, 82.0), turned to 180 degrees
- moved C34 219.4 mm to (49.8, 84.4), turned to 90 degrees
- moved R27 219.2 mm to (49.8, 87.4), turned to -90 degrees
- moved R80 149.3 mm to (65.4, 52.4)
- moved R1 147.5 mm to (59.4, 56.0), turned to -90 degrees
- moved R37 144.6 mm to (48.3, 95.4), turned to 90 degrees
- moved R38 144.2 mm to (49.8, 95.4), turned to 90 degrees
- moved D2 143.4 mm to (54.7, 77.5)
- moved C1 141.5 mm to (61.0, 56.0), turned to 90 degrees
- moved R2 140.5 mm to (59.8, 71.6)
- moved C6 140.5 mm to (73.3, 51.5), turned to -90 degrees
- moved U1 139.5 mm to (59.5, 78.4), turned to 90 degrees
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Connections:
- net /12V_5V/5V_OUT renamed /+5V
- net /RS485_ESP32/RS485_A renamed /RS485_ESP32/RS485_P
- net /RS485_ESP32/RS485_B renamed /RS485_ESP32/RS485_N
- CN10 pad 1: Net-(CN10-Pad1) -> /LED灯驱动2/LED_Drain
- CN10 pad 2: /LED灯驱动2/LED_Drain -> Net-(CN10-Pad2)
- CN8 pad 1: Net-(CN8-Pad1) -> /LED灯驱动/LED_Drain
- CN8 pad 2: /LED灯驱动/LED_Drain -> Net-(CN8-Pad2)
- CN9 pad 1: Net-(CN9-Pad1) -> /LED灯驱动1/LED_Drain
- CN9 pad 2: /LED灯驱动1/LED_Drain -> Net-(CN9-Pad2)
- SW2 pad 2: /ESP32_BOOT -> /GND
- SW2 pad 4: /GND -> /ESP32_BOOT
- U4 pad 2: Net-(CN8-Pad1) -> Net-(CN8-Pad2)
- U5 pad 2: Net-(CN9-Pad1) -> Net-(CN9-Pad2)
- U6 pad 2: Net-(CN10-Pad1) -> Net-(CN10-Pad2)
Routing:
- net /E_STOP: track 0.00 -> 74.5 mm, vias 0 -> 1
- net /+3V3: track 25.0 -> 84.2 mm, vias 2 -> 12
- net /GND: track 32.9 -> 91.0 mm, vias 20 -> 32
- net /RS485_ESP32/RS485_N: track 0.00 -> 46.6 mm
- net /RS485_ESP32/RS485_P: track 0.00 -> 42.4 mm, vias 0 -> 2
- net /RS485_ESP32/RS485_TX: track 0.00 -> 27.5 mm, vias 0 -> 2
- net /RS485_DE: track 0.00 -> 23.2 mm, vias 0 -> 2
- net /RS485_ESP32/RS485_RX: track 0.00 -> 21.3 mm
- net /ESP32_BOOT: track 0.00 -> 18.8 mm, vias 0 -> 2
- net /ESP32_EN: track 0.00 -> 18.5 mm, vias 0 -> 2
- net Net-(U1-EN): track 0.00 -> 8.09 mm
- net /3V3_5V_转换器/5V_SIG0: track 0.00 -> 7.54 mm
- net /+12V: track 10.2 -> 17.6 mm, vias 11 -> 10
- net /3V3_5V_转换器/5V_SIG2: track 0.00 -> 7.40 mm
- net /3V3_5V_转换器/5V_SIG1: track 0.00 -> 6.38 mm
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- added copper zone on B.Cu, net /+12V
- added copper zone on B.Cu, net /+3V3
- added copper zone on B.Cu, net /GND
- added copper zone on F.Cu, net /LED灯驱动/LED_Drain
- added copper zone on B.Cu, net /LED灯驱动1/LED_Drain
- added copper zone on F.Cu, net /LED灯驱动1/LED_Drain
- added copper zone on B.Cu, net /LED灯驱动2/LED_Drain
- added copper zone on F.Cu, net /LED灯驱动2/LED_Drain
- added copper zone on F.Cu, net Net-(CN2-Pad3)
- added copper zone on F.Cu, net Net-(CN3-Pad3)
- added copper zone on F.Cu, net Net-(F1-Pad1)
- added copper zone on B.Cu, net Net-(U10-SW)
- added copper zone on B.Cu, net Net-(U11-SW)
- removed copper zone on In1.Cu, net /GND
- removed copper zone on In2.Cu, net Net-(U10-SW)
- removed copper zone on In2.Cu, net Net-(U11-SW)
Other:
- board size 105 x 90 mm -> 51 x 87.5 mm
- copper layers 4 -> 2
