File: overbed_table/12V_5V.kicad_sch (KiCad schematic)
At the start: 9 parts, among them U2 TPS562201DDCR

Commit message: 原理图V1.0
Parts:
- removed L2: 3.3uH, symbol Device:L
- added L2: FXL0630-3R3-M, lcsc_footprints:C167219_IND-SMD_L7_0-W6_6, symbol lcsc_imported:FXL0630-3R3-M
- C14: renamed from C7; footprint (none) -> Capacitor_SMD:C_0805_2012Metric; 耐压 (none) -> 25V
- C15: renamed from C8; footprint (none) -> Capacitor_SMD:C_0805_2012Metric; 耐压 (none) -> 25V
- C16: renamed from C11; footprint (none) -> Capacitor_SMD:C_0805_2012Metric; 耐压 (none) -> 25V
- C17: renamed from C9; footprint (none) -> Capacitor_SMD:C_0805_2012Metric; 耐压 (none) -> 10V
- C18: renamed from C10; footprint (none) -> Capacitor_SMD:C_0805_2012Metric; 耐压 (none) -> 10V
- R10: renamed from R2; footprint (none) -> Resistor_SMD:R_0603_1608Metric
- R9: renamed from R1; footprint lcsc_footprints:C90061_SOT-23-6_L2_9-W1_6-P0_95-LS2_8-BR -> Resistor_SMD:R_0603_1608Metric
- renumbered U2 to U11
Connections:
- net 5V_OUT: now also L2.2
- net at C16.2, U11.2 (SW): now also L2.1
Other:
- moved on the sheet: R9

Commit message: update: 更新主板电源指示灯
Parts:
- added D5: LED, LED_SMD:LED_0603_1608Metric, symbol Device:LED
- added R20: 4.7k, Resistor_SMD:R_0603_1608Metric, symbol PCM_SparkFun-Resistor:R
Connections:
- net 5V_OUT: now also D5.2 (A)
- net GND: now also R20.1
- new net: D5.1 (K), R20.2

Commit message: update: 添加主板测试点
Parts:
- added TP1: TestPoint, TestPoint:TestPoint_Pad_D2.5mm, symbol Connector:TestPoint
Connections:
- net 5V_OUT: now also TP1.1
Changed lines of the file:
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@@
 	(paper "A4")
 	(junction
+		(at 229.87 72.39)
+		(diameter 0)
+		(color 0 0 0 0)
+	)
+	(junction
 		(at 91.44 72.39)
 		(diameter 0)
@@
 	(wire
 		(pts
+			(xy 229.87 72.39) (xy 236.22 72.39)
+		)
+		(stroke
+			(width 0)
+			(type default)
+		)
+	)
+	(wire
+		(pts
 			(xy 80.01 72.39) (xy 91.44 72.39)
 		)
@@
 	(wire
 		(pts
-			(xy 223.52 72.39) (xy 236.22 72.39)
+			(xy 223.52 72.39) (xy 229.87 72.39)
 		)
 		(stroke
@@
 					(unit 1)
 				)
+			)
+		)
+	)
+	(symbol
+		(lib_id "Connector:TestPoint")
+		(at 229.87 72.39 0)
+		(unit 1)
+		(body_style 1)
+		(exclude_from_sim no)
+		(in_bom yes)
+		(on_board yes)
+		(in_pos_files yes)
+		(dnp no)
+		(fields_autoplaced yes)
+		(property "Reference" "TP1"
+			(at 232.41 67.8179 0)
+			(show_name no)
+			(do_not_autoplace no)
+			(effects
+				(font
+					(size 1.27 1.27)
+				)
+				(justify left)
+			)
+		)
+		(property "Value" "TestPoint"
+			(at 232.41 70.3579 0)
+			(show_name no)
+			(do_not_autoplace no)
+			(effects
+				(font
+					(size 1.27 1.27)
+				)
+				(justify left)
+			)
+		)
+		(property "Footprint" "TestPoint:TestPoint_Pad_D2.5mm"
+			(at 234.95 72.39 0)
+			(hide yes)
+			(show_name no)
+			(do_not_autoplace no)
+			(effects
+				(font
+					(size 1.27 1.27)
+				)
+			)
+		)
+		(property "Datasheet" ""
+			(at 234.95 72.39 0)
+			(hide yes)
+			(show_name no)
+			(do_not_autoplace no)
+			(effects
+				(font
+					(size 1.27 1.27)
+				)
+			)
+		)
+		(property "Description" "test point"
+			(at 229.87 72.39 0)
+			(hide yes)
+			(show_name no)
+			(do_not_autoplace no)
+			(effects
+				(font
+					(size 1.27 1.27)
+				)
+			)
+		)
+		(pin "1"
+		)
+		(instances
+			(project "overbed_table"
+				(path "/ea72387d-aa38-4027-b8fe-1f6fcfee6654/ebc9d23c-4131-4c15-866f-2eb222d4508c"
+					(reference "TP1")
+					(unit 1)
+				)
