File: overbed_table/_restore_backup_2026-09-04T14-28-33-293/步进驱动.kicad_sch (KiCad schematic)
At the start: 23 parts, among them U4 TMC2209-LA

Commit message: 更新步进驱动等
Parts:
- removed C21: C, Display_7Segment:HDSP-7401, symbol Device:C
- removed C22, C23: 100nF, Display_7Segment:HDSP-7401, symbol Device:C
- removed C24: 100uF, Display_7Segment:HDSP-7401, symbol Device:C
- removed TP10, TP2, TP3, TP4, TP5, TP6, TP7, TP8, TP9: TestPoint, symbol Connector:TestPoint
Connections:
- net at U4.17 (VREF): no longer TP1.1
