File: side_panel/RS485_PY32.kicad_sch (KiCad schematic)
At the start: 4 parts, among them U35 SP3485EN

Commit message: 更新针脚变动
Parts:
- R18: renamed from R76; footprint PCM_SparkFun-Resistor:R_0603_1608Metric -> Resistor_SMD:R_0603_1608Metric
- R19: renamed from R77; footprint PCM_SparkFun-Resistor:R_0603_1608Metric -> Resistor_SMD:R_0603_1608Metric
- renumbered C78 to C15, U35 to U8
Changed lines of the file:
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@@
 		(dnp no)
 		(fields_autoplaced yes)
-		(property "Reference" "C78"
+		(property "Reference" "C15"
 			(at 143.51 59.69 90)
 			(show_name no)
@@
 			(project "side_panel"
 				(path "/6f325c3b-cf1b-4cbd-9ec7-aa44385f0008/dcc0c29f-55e6-46e1-9fee-927044492ad7"
-					(reference "C78")
+					(reference "C15")
 					(unit 1)
 				)
@@
 		(dnp no)
 		(fields_autoplaced yes)
-		(property "Reference" "R76"
+		(property "Reference" "R18"
 			(at 97.79 93.9799 90)
 			(show_name no)
@@
 			)
 		)
-		(property "Footprint" "PCM_SparkFun-Resistor:R_0603_1608Metric"
+		(property "Footprint" "Resistor_SMD:R_0603_1608Metric"
 			(at 99.822 95.25 0)
 			(hide yes)
@@
 			(project "side_panel"
 				(path "/6f325c3b-cf1b-4cbd-9ec7-aa44385f0008/dcc0c29f-55e6-46e1-9fee-927044492ad7"
-					(reference "R76")
+					(reference "R18")
 					(unit 1)
 				)
@@
 		(dnp no)
 		(fields_autoplaced yes)
-		(property "Reference" "U35"
+		(property "Reference" "U8"
 			(at 136.7633 71.12 0)
 			(show_name no)
@@
 			(project "side_panel"
 				(path "/6f325c3b-cf1b-4cbd-9ec7-aa44385f0008/dcc0c29f-55e6-46e1-9fee-927044492ad7"
-					(reference "U35")
+					(reference "U8")
 					(unit 1)
 				)
@@
 		(dnp no)
 		(fields_autoplaced yes)
-		(property "Reference" "R77"
+		(property "Reference" "R19"
 			(at 163.83 82.5499 90)
 			(show_name no)
@@
 			)
 		)
-		(property "Footprint" "PCM_SparkFun-Resistor:R_0603_1608Metric"
+		(property "Footprint" "Resistor_SMD:R_0603_1608Metric"
 			(at 165.862 83.82 0)
 			(hide yes)
@@
 			(project "side_panel"
 				(path "/6f325c3b-cf1b-4cbd-9ec7-aa44385f0008/dcc0c29f-55e6-46e1-9fee-927044492ad7"
-					(reference "R77")
+					(reference "R19")
 					(unit 1)
 				)
