File: side_panel/TOF.kicad_sch (KiCad schematic)
At the start: 9 parts, among them U32 VL53L0CXV0DH1

Commit message: 更新针脚变动
Parts:
- R20: renamed from R69; footprint PCM_SparkFun-Resistor:R_0603_1608Metric -> Resistor_SMD:R_0603_1608Metric
- R21: renamed from R70; footprint PCM_SparkFun-Resistor:R_0603_1608Metric -> Resistor_SMD:R_0603_1608Metric
- R22: renamed from R71; footprint PCM_SparkFun-Resistor:R_0603_1608Metric -> Resistor_SMD:R_0603_1608Metric
- renumbered C68 to C16, C69 to C17, TP32 to TP1, TP33 to TP2, TP34 to TP3, U32 to U9
Changed lines of the file:
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@@
 		(dnp no)
 		(fields_autoplaced yes)
-		(property "Reference" "#PWR0141"
+		(property "Reference" "#PWR041"
 			(at 63.5 158.75 0)
 			(hide yes)
@@
 			(project "side_panel"
 				(path "/6f325c3b-cf1b-4cbd-9ec7-aa44385f0008/c9bb3357-dcaa-4211-b368-89a3c1409a9c"
-					(reference "#PWR0141")
+					(reference "#PWR041")
 					(unit 1)
 				)
@@
 		(dnp no)
 		(fields_autoplaced yes)
-		(property "Reference" "C68"
+		(property "Reference" "C16"
 			(at 46.99 138.4299 0)
 			(show_name no)
@@
 			(project "side_panel"
 				(path "/6f325c3b-cf1b-4cbd-9ec7-aa44385f0008/c9bb3357-dcaa-4211-b368-89a3c1409a9c"
-					(reference "C68")
+					(reference "C16")
 					(unit 1)
 				)
@@
 		(dnp no)
 		(fields_autoplaced yes)
-		(property "Reference" "R69"
+		(property "Reference" "R20"
 			(at 99.06 91.4399 90)
 			(show_name no)
@@
 			)
 		)
-		(property "Footprint" "PCM_SparkFun-Resistor:R_0603_1608Metric"
+		(property "Footprint" "Resistor_SMD:R_0603_1608Metric"
 			(at 101.092 92.71 0)
 			(hide yes)
@@
 			(project "side_panel"
 				(path "/6f325c3b-cf1b-4cbd-9ec7-aa44385f0008/c9bb3357-dcaa-4211-b368-89a3c1409a9c"
-					(reference "R69")
+					(reference "R20")
 					(unit 1)
 				)
@@
 		(dnp no)
 		(fields_autoplaced yes)
-		(property "Reference" "C69"
+		(property "Reference" "C17"
 			(at 60.96 138.4299 0)
 			(show_name no)
@@
 			(project "side_panel"
 				(path "/6f325c3b-cf1b-4cbd-9ec7-aa44385f0008/c9bb3357-dcaa-4211-b368-89a3c1409a9c"
-					(reference "C69")
+					(reference "C17")
 					(unit 1)
 				)
@@
 	)
 	(symbol
-		(lib_name "GND_1")
 		(lib_id "power:GND")
 		(at 134.62 128.27 0)
@@
 		(dnp no)
 		(fields_autoplaced yes)
-		(property "Reference" "#PWR0143"
+		(property "Reference" "#PWR043"
 			(at 134.62 134.62 0)
 			(hide yes)
@@
 			(project "side_panel"
 				(path "/6f325c3b-cf1b-4cbd-9ec7-aa44385f0008/c9bb3357-dcaa-4211-b368-89a3c1409a9c"
-					(reference "#PWR0143")
+					(reference "#PWR043")
 					(unit 1)
 				)
@@
 		(dnp no)
 		(fields_autoplaced yes)
-		(property "Reference" "U32"
+		(property "Reference" "U9"
 			(at 143.51 100.3299 0)
 			(show_name no)
@@
 			(project "side_panel"
 				(path "/6f325c3b-cf1b-4cbd-9ec7-aa44385f0008/c9bb3357-dcaa-4211-b368-89a3c1409a9c"
-					(reference "U32")
+					(reference "U9")
 					(unit 1)
 				)
@@
 		(dnp no)
 		(fields_autoplaced yes)
-		(property "Reference" "TP34"
+		(property "Reference" "TP3"
 			(at 119.38 87.63 0)
 			(show_name no)
@@
 			(project "side_panel"
 				(path "/6f325c3b-cf1b-4cbd-9ec7-aa44385f0008/c9bb3357-dcaa-4211-b368-89a3c1409a9c"
-					(reference "TP34")
+					(reference "TP3")
 					(unit 1)
 				)
@@
 		(dnp no)
 		(fields_autoplaced yes)
-		(property "Reference" "TP32"
+		(property "Reference" "TP1"
 			(at 80.01 93.98 0)
 			(show_name no)
@@
 			(project "side_panel"
 				(path "/6f325c3b-cf1b-4cbd-9ec7-aa44385f0008/c9bb3357-dcaa-4211-b368-89a3c1409a9c"
-					(reference "TP32")
+					(reference "TP1")
 					(unit 1)
 				)
@@
 		(dnp no)
 		(fields_autoplaced yes)
-		(property "Reference" "#PWR0140"
+		(property "Reference" "#PWR040"
 			(at 63.5 130.81 0)
 			(hide yes)
@@
 			(project "side_panel"
 				(path "/6f325c3b-cf1b-4cbd-9ec7-aa44385f0008/c9bb3357-dcaa-4211-b368-89a3c1409a9c"
-					(reference "#PWR0140")
+					(reference "#PWR040")
 					(unit 1)
 				)
@@
 		(dnp no)
 		(fields_autoplaced yes)
-		(property "Reference" "#PWR0142"
+		(property "Reference" "#PWR042"
 			(at 134.62 80.01 0)
 			(hide yes)
@@
 			(project "side_panel"
 				(path "/6f325c3b-cf1b-4cbd-9ec7-aa44385f0008/c9bb3357-dcaa-4211-b368-89a3c1409a9c"
-					(reference "#PWR0142")
+					(reference "#PWR042")
 					(unit 1)
 				)
@@
 		(dnp no)
 		(fields_autoplaced yes)
-		(property "Reference" "R70"
+		(property "Reference" "R21"
 			(at 109.22 91.4399 90)
 			(show_name no)
@@
 			)
 		)
-		(property "Footprint" "PCM_SparkFun-Resistor:R_0603_1608Metric"
+		(property "Footprint" "Resistor_SMD:R_0603_1608Metric"
 			(at 111.252 92.71 0)
 			(hide yes)
@@
 			(project "side_panel"
 				(path "/6f325c3b-cf1b-4cbd-9ec7-aa44385f0008/c9bb3357-dcaa-4211-b368-89a3c1409a9c"
-					(reference "R70")
+					(reference "R21")
 					(unit 1)
 				)
@@
 		(dnp no)
 		(fields_autoplaced yes)
-		(property "Reference" "R71"
+		(property "Reference" "R22"
 			(at 121.92 116.8399 90)
 			(show_name no)
@@
 			)
 		)
-		(property "Footprint" "PCM_SparkFun-Resistor:R_0603_1608Metric"
+		(property "Footprint" "Resistor_SMD:R_0603_1608Metric"
 			(at 123.952 118.11 0)
 			(hide yes)
@@
 			(project "side_panel"
 				(path "/6f325c3b-cf1b-4cbd-9ec7-aa44385f0008/c9bb3357-dcaa-4211-b368-89a3c1409a9c"
-					(reference "R71")
+					(reference "R22")
 					(unit 1)
 				)
@@
 		(dnp no)
 		(fields_autoplaced yes)
-		(property "Reference" "TP33"
+		(property "Reference" "TP2"
 			(at 88.9 93.98 0)
 			(show_name no)
@@
 			(project "side_panel"
 				(path "/6f325c3b-cf1b-4cbd-9ec7-aa44385f0008/c9bb3357-dcaa-4211-b368-89a3c1409a9c"
-					(reference "TP33")
+					(reference "TP2")
 					(unit 1)
 				)
