File: side_panel/升降电机驱动.kicad_sch (KiCad schematic)
At the start: 5 parts, among them U34 SS6285M-SO-TP

Commit message: 更新针脚变动
Parts:
- R23: renamed from R74; footprint PCM_SparkFun-Resistor:R_0603_1608Metric -> Resistor_SMD:R_0603_1608Metric
- R24: renamed from R75; footprint PCM_SparkFun-Resistor:R_0603_1608Metric -> Resistor_SMD:R_0603_1608Metric
- renumbered C76 to C18, C77 to C19, U34 to U10
Changed lines of the file:
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@@
 		(dnp no)
 		(fields_autoplaced yes)
-		(property "Reference" "#PWR0146"
+		(property "Reference" "#PWR046"
 			(at 114.3 36.83 0)
 			(hide yes)
@@
 			(project "side_panel"
 				(path "/6f325c3b-cf1b-4cbd-9ec7-aa44385f0008/d466b5a9-aa1a-4f39-ad33-b77ddb4cccb3"
-					(reference "#PWR0146")
+					(reference "#PWR046")
 					(unit 1)
 				)
@@
 		(dnp no)
 		(fields_autoplaced yes)
-		(property "Reference" "C76"
+		(property "Reference" "C18"
 			(at 82.55 64.7699 0)
 			(show_name no)
@@
 			(project "side_panel"
 				(path "/6f325c3b-cf1b-4cbd-9ec7-aa44385f0008/d466b5a9-aa1a-4f39-ad33-b77ddb4cccb3"
-					(reference "C76")
+					(reference "C18")
 					(unit 1)
 				)
@@
 		(dnp no)
 		(fields_autoplaced yes)
-		(property "Reference" "#PWR0148"
+		(property "Reference" "#PWR048"
 			(at 134.62 71.12 0)
 			(hide yes)
@@
 			(project "side_panel"
 				(path "/6f325c3b-cf1b-4cbd-9ec7-aa44385f0008/d466b5a9-aa1a-4f39-ad33-b77ddb4cccb3"
-					(reference "#PWR0148")
+					(reference "#PWR048")
 					(unit 1)
 				)
@@
 		(dnp yes)
 		(fields_autoplaced yes)
-		(property "Reference" "R75"
+		(property "Reference" "R24"
 			(at 134.62 52.0699 90)
 			(show_name no)
@@
 			)
 		)
-		(property "Footprint" "PCM_SparkFun-Resistor:R_0603_1608Metric"
+		(property "Footprint" "Resistor_SMD:R_0603_1608Metric"
 			(at 136.652 53.34 0)
 			(hide yes)
@@
 			(project "side_panel"
 				(path "/6f325c3b-cf1b-4cbd-9ec7-aa44385f0008/d466b5a9-aa1a-4f39-ad33-b77ddb4cccb3"
-					(reference "R75")
+					(reference "R24")
 					(unit 1)
 				)
@@
 		(dnp no)
 		(fields_autoplaced yes)
-		(property "Reference" "C77"
+		(property "Reference" "C19"
 			(at 97.79 63.8809 0)
 			(show_name no)
@@
 			(project "side_panel"
 				(path "/6f325c3b-cf1b-4cbd-9ec7-aa44385f0008/d466b5a9-aa1a-4f39-ad33-b77ddb4cccb3"
-					(reference "C77")
+					(reference "C19")
 					(unit 1)
 				)
@@
 		(dnp yes)
 		(fields_autoplaced yes)
-		(property "Reference" "R74"
+		(property "Reference" "R23"
 			(at 116.84 55.8799 90)
 			(show_name no)
@@
 			)
 		)
-		(property "Footprint" "PCM_SparkFun-Resistor:R_0603_1608Metric"
+		(property "Footprint" "Resistor_SMD:R_0603_1608Metric"
 			(at 118.872 57.15 0)
 			(hide yes)
@@
 			(project "side_panel"
 				(path "/6f325c3b-cf1b-4cbd-9ec7-aa44385f0008/d466b5a9-aa1a-4f39-ad33-b77ddb4cccb3"
-					(reference "R74")
+					(reference "R23")
 					(unit 1)
 				)
@@
 		(dnp no)
 		(fields_autoplaced yes)
-		(property "Reference" "#PWR0144"
+		(property "Reference" "#PWR044"
 			(at 93.98 57.15 0)
 			(hide yes)
@@
 			(project "side_panel"
 				(path "/6f325c3b-cf1b-4cbd-9ec7-aa44385f0008/d466b5a9-aa1a-4f39-ad33-b77ddb4cccb3"
-					(reference "#PWR0144")
+					(reference "#PWR044")
 					(unit 1)
 				)
@@
 		(dnp no)
 		(fields_autoplaced yes)
-		(property "Reference" "U34"
+		(property "Reference" "U10"
 			(at 149.86 53.34 0)
 			(show_name no)
@@
 			(project "side_panel"
 				(path "/6f325c3b-cf1b-4cbd-9ec7-aa44385f0008/d466b5a9-aa1a-4f39-ad33-b77ddb4cccb3"
-					(reference "U34")
+					(reference "U10")
 					(unit 1)
 				)
@@
 	)
 	(symbol
-		(lib_name "GND_2")
 		(lib_id "power:GND")
 		(at 124.46 76.2 0)
@@
 		(dnp no)
 		(fields_autoplaced yes)
-		(property "Reference" "#PWR0147"
+		(property "Reference" "#PWR047"
 			(at 124.46 82.55 0)
 			(hide yes)
@@
 			(project "side_panel"
 				(path "/6f325c3b-cf1b-4cbd-9ec7-aa44385f0008/d466b5a9-aa1a-4f39-ad33-b77ddb4cccb3"
-					(reference "#PWR0147")
+					(reference "#PWR047")
 					(unit 1)
 				)
@@
 	)
 	(symbol
-		(lib_name "GND_1")
 		(lib_id "power:GND")
 		(at 93.98 78.74 0)
@@
 		(dnp no)
 		(fields_autoplaced yes)
-		(property "Reference" "#PWR0145"
+		(property "Reference" "#PWR045"
 			(at 93.98 85.09 0)
 			(hide yes)
@@
 			(project "side_panel"
 				(path "/6f325c3b-cf1b-4cbd-9ec7-aa44385f0008/d466b5a9-aa1a-4f39-ad33-b77ddb4cccb3"
-					(reference "#PWR0145")
+					(reference "#PWR045")
 					(unit 1)
 				)
