File: side_panel/步进驱动.kicad_sch (KiCad schematic)
At the start: 23 parts, among them U31 TMC2209-LA

Commit message: feat: 添加侧电机板基础元件布局
Parts:
- removed TP24, TP25: TestPoint, PCM_SparkFun-Connector:TestPoint-1.0mm, symbol Connector:TestPoint

Commit message: 更新针脚变动
Parts:
- R25: renamed from R65; footprint PCM_SparkFun-Resistor:R_0603_1608Metric -> Resistor_SMD:R_0603_1608Metric
- R26: renamed from R66; footprint PCM_SparkFun-Resistor:R_0603_1608Metric -> Resistor_SMD:R_0603_1608Metric
- R27: renamed from R67; footprint Resistor_SMD:R_1206_3216Metric -> Resistor_SMD:R_0603_1608Metric
- R28: renamed from R68; footprint Resistor_SMD:R_1206_3216Metric -> Resistor_SMD:R_0603_1608Metric
- renumbered C60 to C20, C61 to C21, C62 to C22, C63 to C23, C64 to C24, C65 to C25, C66 to C26, C67 to C27, TP30 to TP10, TP31 to TP11, TP22 to TP4, TP23 to TP5, TP26 to TP6, TP27 to TP7, TP28 to TP8, TP29 to TP9, U31 to U11
